Commit message: update bagian kinematic dan wheel transmission xacro nya dan swerve drive urdf xacro dan joystick.yaml nya

File: install/swerve_description/share/swerve_description/urdf/base/base.gazebo.xacro (robot description, xacro)
@@ -1,10 +1 @@
-<?xml version="1.0"?>
-<robot xmlns:xacro="http://ros.org/wiki/xacro">
-  <xacro:macro name="base_gazebo_v0" params= "link_name">
-    <gazebo reference="${link_name}">
-      <selfCollide>false</selfCollide>
-      <mu1 value="0.05" />
-      <mu2 value="0.05" />
-    </gazebo>
-  </xacro:macro>
-</robot>
+/home/syafihidayat/swerve_test/src/swerve_description/urdf/base/base.gazebo.xacro

File: install/swerve_description/share/swerve_description/urdf/base/base.urdf.xacro (robot description, xacro)
@@ -1,36 +1 @@
-<?xml version="1.0"?>
-<robot xmlns:xacro="http://ros.org/wiki/xacro">
-	<xacro:include filename="$(find swerve_description)/urdf/common.xacro"/>
-	<xacro:include filename="$(find swerve_description)/urdf/base/base.gazebo.xacro"/>
-	<xacro:property name="base_height" value="0.15"/>
-    <xacro:property name="base_width" value="0.09"/>
-    <xacro:property name="base_depth" value="0.015"/>
-    <xacro:property name="base_mass" value="0.5"/>
-	<xacro:macro name="base_v0" params="link_name parent *joint_origin">
-		<joint name="${link_name}_joint" type="fixed">
-			<xacro:insert_block name="joint_origin"/>
-			<parent link="${parent}"/>
-			<child link="${link_name}"/>
-		</joint>
-		<link name="${link_name}">
-			<visual>
-				<geometry>
-					<!-- <mesh filename="package://swerve_description/meshes/stl/base.STL"/> -->
-					<box size="0.15 0.09 0.015"/>
-				</geometry>
-				<origin xyz="0 0 0" />
-				<material name="gray"/>
-			</visual>
-			<collision>
-				<geometry>
-					<box size="${base_height} ${base_width} ${base_depth}"/>
-				</geometry>
-				<origin xyz="0 0 ${base_depth/2}" />
-			</collision>
-			<inertial>
-				<origin xyz="0 0 ${base_depth/2}"/>
-				<xacro:box_inertial mass="${base_mass}" height="${base_height}" width="${base_width}" depth="${base_depth}"/>
-			</inertial>
-		</link>
-	</xacro:macro>
-</robot>
+/home/syafihidayat/swerve_test/src/swerve_description/urdf/base/base.urdf.xacro

File: install/swerve_description/share/swerve_description/urdf/color_palette.xacro (robot description, xacro)
@@ -1,13 +1 @@
-<?xml version="1.0"?>
-<robot xmlns:xacro="http://ros.org/wiki/xacro">
-    <material name="green">
-        <color rgba="0 0.7 0 1"/>
-    </material>
-    <material name="gray">
-		<!-- <color rgba="0.5 0.5 0.5 2.5"/> -->
-    <color rgba="0.5 0.5 0.5 1.0"/>
-    </material>
-    <material name="blue">
-		<color rgba="0 0 1 1"/>
-	</material>
-</robot>
+/home/syafihidayat/swerve_test/src/swerve_description/urdf/color_palette.xacro

File: install/swerve_description/share/swerve_description/urdf/common.xacro (robot description, xacro)
@@ -1,12 +1 @@
-<?xml version="1.0"?>
-<robot xmlns:xacro="http://ros.org/wiki/xacro">
-    <xacro:property name="M_PI" value="3.14159274"/>
-    <xacro:macro name="cylinder_inertial" params="mass radius length">
-        <mass value="${mass}"/>
-        <inertia ixx="${((radius*radius)/4 + (length*length)/12)*mass}" ixy="0" ixz="0" iyy="${((radius*radius)/4 + (length*length)/12)*mass}" iyz="0" izz="${(mass*radius*radius)/2}" />
-    </xacro:macro>
-    <xacro:macro name="box_inertial" params="mass height width depth">
-        <mass value="${mass}"/>
-        <inertia ixx="${(mass*(width*width+depth*depth))/12}" ixy="0" ixz="0" iyy="${(mass*(height*height+depth*depth))/12}" iyz="0" izz="${(mass*(height*height+width*width))/12}" />
-    </xacro:macro>
-</robot>
+/home/syafihidayat/swerve_test/src/swerve_description/urdf/common.xacro

File: install/swerve_description/share/swerve_description/urdf/swerve_drive/steering.transmission.xacro (robot description, xacro)
@@ -1,27 +1 @@
-<?xml version="1.0"?>
-<robot xmlns:xacro="http://ros.org/wiki/xacro">
-    <xacro:macro name="steering_trans_v0" params="prefix">
-        <ros2_control name="${prefix}_steering_system" type="system">
-            <hardware>
-                <plugin>gazebo_ros2_control/GazeboSystem</plugin>
-            </hardware>
-            <joint name="${prefix}_steering_joint">
-                <command_interface name="velocity"/>
-                <state_interface name="position"/>
-                <state_interface name="velocity"/>
-            </joint>
-        </ros2_control>
-    </xacro:macro>
-    <!-- <xacro:macro name="steering_trans_v0" params="prefix">
-        <ros2_control name="${prefix}_steering_system" type="system">
-            <hardware>
-                <plugin>gazebo_ros2_control/GazeboSystem</plugin>
-            </hardware>
-            <joint name="${prefix}_steering_joint">
-                <command_interface name="position"/>
-                <state_interface name="position"/>
-                <state_interface name="velocity"/>
-            </joint>
-        </ros2_control>
-    </xacro:macro> -->
-</robot>
+/home/syafihidayat/swerve_test/src/swerve_description/urdf/swerve_drive/steering.transmission.xacro

File: install/swerve_description/share/swerve_description/urdf/swerve_drive/swerve_drive.gazebo.xacro (robot description, xacro)
@@ -1,21 +1 @@
-<?xml version="1.0"?>
-<robot xmlns:xacro="http://ros.org/wiki/xacro">
-    <xacro:macro name="swerve_drive_gazebo_v0" params="prefix">
-        <!-- steering-->
-        <gazebo reference="${prefix}_steering_link">
-            <selfCollide>false</selfCollide>
-            <mu1 value="0.4" />
-            <mu2 value="0.4" />
-            <kp>1e8</kp>
-            <kd>1e8</kd>
-        </gazebo>
-        <!-- wheel-->
-        <gazebo reference="${prefix}_wheel_link">
-            <selfCollide>false</selfCollide>
-            <mu1 value="0.4" />
-            <mu2 value="0.4" />
-            <kp>1e8</kp>
-            <kd>1e8</kd>
-        </gazebo>
-    </xacro:macro>
-</robot>
+/home/syafihidayat/swerve_test/src/swerve_description/urdf/swerve_drive/swerve_drive.gazebo.xacro

File: install/swerve_description/share/swerve_description/urdf/swerve_drive/swerve_drive.urdf.xacro (robot description, xacro)
@@ -1,72 +1 @@
-<?xml version="1.0"?>
-<robot xmlns:xacro="http://ros.org/wiki/xacro">
-    <xacro:include filename="$(find swerve_description)/urdf/common.xacro"/>
-    <xacro:include filename="$(find swerve_description)/urdf/swerve_drive/steering.transmission.xacro"/>
-    <xacro:include filename="$(find swerve_description)/urdf/swerve_drive/wheel.transmission.xacro"/>
-    <xacro:include filename="$(find swerve_description)/urdf/swerve_drive/swerve_drive.gazebo.xacro"/>
-    <xacro:property name="steering_radius" value="0.015"/>
-    <xacro:property name="steering_length" value="0.003"/>
-    <xacro:property name="steering_mass" value="0.01"/>
-    <xacro:property name="wheel_radius" value="0.01"/>
-    <xacro:property name="wheel_length" value="0.01"/>
-    <xacro:property name="wheel_mass" value="0.05"/>
-    <xacro:macro name="swerve_drive_v0" params="prefix parent *joint_origin *joint_axis_s *joint_axis_w">
-        <!-- steering -->
-        <joint name="${prefix}_steering_joint" type="revolute">
-            <xacro:insert_block name="joint_origin"/>
-            <parent link="${parent}"/>
-            <child link="${prefix}_steering_link"/>
-            <xacro:insert_block name="joint_axis_s"/>
-            <limit lower="-${M_PI}" upper="${M_PI}" effort="10" velocity="10"/>
-        </joint>
-        <link name="${prefix}_steering_link">
-            <visual>
-                <geometry>
-                    <mesh filename="package://swerve_description/meshes/dae/steering.dae"/>
-                    <!-- <cylinder radius="${steering_radius}" length="${steering_length}"/> -->
-                </geometry>
-                <origin xyz="0 0 0" />
-                <material name="blue"/>
-            </visual>
-            <collision>
-                <geometry>
-                    <cylinder radius="${steering_radius}" length="${steering_length}"/>
-                </geometry>
-                <origin xyz="0 0 ${steering_length/2}"/>
-            </collision>
-            <inertial>
-                <origin xyz="0 0 ${steering_length/2}"/>
-                <xacro:cylinder_inertial mass="${steering_mass}" radius="${steering_radius}" length="${steering_length}"/>
-            </inertial>
-        </link>
-        <!-- wheel -->
-        <joint name="${prefix}_wheel_joint" type="continuous">
-            <origin xyz="0 0 0.005"/>
-            <parent link="${prefix}_steering_link"/>
-            <child link="${prefix}_wheel_link"/>
-            <xacro:insert_block name="joint_axis_w"/>
-            <limit velocity="15.0" effort="0.001" />
-            <dynamics damping="0"/>
-        </joint>
-        <link name="${prefix}_wheel_link">
-            <visual>
-                <geometry>
-                    <mesh filename="package://swerve_description/meshes/dae/wheel.dae"/>
-                    <!-- <cylinder radius="${steering_radius}" length="${steering_length}"/> -->
-                </geometry>
-                <origin xyz="0 -${wheel_length/2} 0"/>
-                <material name="green"/>
-            </visual>
-            <collision>
-                <origin xyz="0 0 0" rpy="${M_PI/2} 0 0"/>
-                <geometry>
-                    <cylinder radius="${wheel_radius}" length="${wheel_length}"/>
-                </geometry>
-            </collision>
-            <inertial>
-                <origin xyz="0 0 0" rpy="${M_PI/2} 0 0"/>
-                <xacro:cylinder_inertial mass="${wheel_mass}" radius="${wheel_radius}" length="${wheel_length}"/>
-            </inertial>
-        </link>
-    </xacro:macro>
-</robot>
+/home/syafihidayat/swerve_test/src/swerve_description/urdf/swerve_drive/swerve_drive.urdf.xacro

File: install/swerve_description/share/swerve_description/urdf/swerve_drive/swerve_drive_robot.urdf.xacro (robot description, xacro)
@@ -1,72 +1 @@
-<?xml version="1.0"?>
-<robot name="swerve_drive_robot" xmlns:xacro="http://ros.org/wiki/xacro">
-    <xacro:include filename="$(find swerve_description)/urdf/color_palette.xacro"/>
-    <xacro:include filename="$(find swerve_description)/urdf/base/base.urdf.xacro"/>
-    <xacro:include filename="$(find swerve_description)/urdf/swerve_drive/swerve_drive.urdf.xacro"/>
-    <xacro:include filename="$(find swerve_description)/urdf/swerve_drive/wheel.transmission.xacro"/>
-    <link name="base_footprint"/>
-    <xacro:base_v0 link_name="base_link" parent="base_footprint">
-		<origin xyz="0 0 0.005"/>
-	</xacro:base_v0>
-	<!-- base_height 0.15 base_length 0.09 steering_radius 0.015-->
-	<!-- Front Right Swerve Drive-->
-	<xacro:swerve_drive_v0 prefix="front_right" parent="base_link">
-		<origin xyz="0.06 -0.06 0" />
-		<!--steering-->
-		<axis xyz="0 0 1"/>
-		<!--wheel-->
-		<axis xyz="0 1 0"/>
-	</xacro:swerve_drive_v0>
-	<!-- Front Left Swerve Drive-->
-	<xacro:swerve_drive_v0 prefix="front_left" parent="base_link">
-		<origin xyz="0.06 0.06 0" />
-		<!--steering-->
-		<axis xyz="0 0 1"/>
-		<!--wheel-->
-		<axis xyz="0 1 0"/>
-	</xacro:swerve_drive_v0>
-	<!-- Rear Right Swerve Drive-->
-	<xacro:swerve_drive_v0 prefix="rear_right" parent="base_link">
-		<origin xyz="-0.06 -0.06 0" />
-		<!--steering-->
-		<axis xyz="0 0 1"/>
-		<!--wheel-->
-		<axis xyz="0 1 0"/>
-	</xacro:swerve_drive_v0>
-	<!-- Rear Left Swerve Drive-->
-	<xacro:swerve_drive_v0 prefix="rear_left" parent="base_link">
-		<origin xyz="-0.06 0.06 0"/>
-		<!--steering-->
-		<axis xyz="0 0 1"/>
-		<!--wheel-->
-		<axis xyz="0 1 0"/>
-	</xacro:swerve_drive_v0>
-	<!-- ===============  Transmission =============== -->
-	<xacro:arg name="load_trans_s" default="true" />
-	<xacro:arg name="load_trans_w" default="true" />
-	<xacro:if value="$(arg load_trans_s)">
-		<xacro:steering_trans_v0 prefix="front_right" />
-		<xacro:steering_trans_v0 prefix="front_left" />
-		<xacro:steering_trans_v0 prefix="rear_right" />
-		<xacro:steering_trans_v0 prefix="rear_left" />
-	</xacro:if>
-	<xacro:if value="$(arg load_trans_w)">
-		<xacro:wheel_trans_v0 prefix="front_right" />
-		<xacro:wheel_trans_v0 prefix="front_left" />
-		<xacro:wheel_trans_v0 prefix="rear_right" />
-		<xacro:wheel_trans_v0 prefix="rear_left" />
-	</xacro:if>
-		<!-- =============== Gazebo =============== -->
-	<!-- Namespace -->
-	<gazebo>
-        <plugin filename="libgazebo_ros2_control.so" name="gazebo_ros2_control">
-            <parameters>$(find swerve_description)/config/controller_steering.yaml</parameters>
-            <parameters>$(find swerve_description)/config/controller_wheel.yaml</parameters>
-        </plugin>
-    </gazebo>
-	<xacro:base_gazebo_v0 link_name="base_link"/>
-	<xacro:swerve_drive_gazebo_v0 prefix="front_right"/>
-	<xacro:swerve_drive_gazebo_v0 prefix="front_left"/>
-	<xacro:swerve_drive_gazebo_v0 prefix="rear_right"/>
-	<xacro:swerve_drive_gazebo_v0 prefix="rear_left"/>
-</robot>
+/home/syafihidayat/swerve_test/src/swerve_description/urdf/swerve_drive/swerve_drive_robot.urdf.xacro

File: install/swerve_description/share/swerve_description/urdf/swerve_drive/wheel.transmission.xacro (robot description, xacro)
@@ -1,27 +1 @@
-<?xml version="1.0"?>
-<robot xmlns:xacro="http://ros.org/wiki/xacro">
-    <xacro:macro name="wheel_trans_v0" params="prefix">
-        <ros2_control name="${prefix}_wheel_system" type="system">
-            <hardware>
-                <plugin>gazebo_ros2_control/GazeboSystem</plugin>
-            </hardware>
-            <joint name="${prefix}_wheel_joint">
-                <command_interface name="effort"/>
-                <state_interface name="position"/>
-                <state_interface name="velocity"/>
-            </joint>
-        </ros2_control>
-    </xacro:macro>
-    <!-- <xacro:macro name="wheel_trans_v0" params="prefix">
-        <ros2_control name="${prefix}_wheel_system" type="system">
-            <hardware>
-                <plugin>gazebo_ros2_control/GazeboSystem</plugin>
-            </hardware>
-            <joint name="${prefix}_wheel_joint">
-                <command_interface name="velocity"/>
-                <state_interface name="position"/>
-                <state_interface name="velocity"/>
-            </joint>
-        </ros2_control>
-    </xacro:macro> -->
-</robot>
+/home/syafihidayat/swerve_test/src/swerve_description/urdf/swerve_drive/wheel.transmission.xacro

File: src/swerve_description/urdf/swerve_drive/swerve_drive.urdf.xacro (robot description, xacro)
@@ -46,5 +46,6 @@
             <child link="${prefix}_wheel_link"/>
             <xacro:insert_block name="joint_axis_w"/>
-            <limit velocity="15.0" effort="0.001" />
+            <limit velocity="15.0" effort="1.0" />
+            <!-- <limit velocity="15.0" effort="0.001" /> -->
             <dynamics damping="0"/>
         </joint>
@@ -62,4 +63,5 @@
                 <geometry>
                     <cylinder radius="${wheel_radius}" length="${wheel_length}"/>
+                    <!-- <cylinder radius="${wheel_radius}" length="${wheel_length}"/> -->
                 </geometry>
             </collision>

File: src/swerve_description/urdf/swerve_drive/wheel.transmission.xacro (robot description, xacro)
@@ -1,5 +1,5 @@
 <?xml version="1.0"?>
 <robot xmlns:xacro="http://ros.org/wiki/xacro">
-    <xacro:macro name="wheel_trans_v0" params="prefix">
+    <!-- <xacro:macro name="wheel_trans_v0" params="prefix">
         <ros2_control name="${prefix}_wheel_system" type="system">
             <hardware>
@@ -12,6 +12,6 @@
             </joint>
         </ros2_control>
-    </xacro:macro>
-    <!-- <xacro:macro name="wheel_trans_v0" params="prefix">
+    </xacro:macro> -->
+    <xacro:macro name="wheel_trans_v0" params="prefix">
         <ros2_control name="${prefix}_wheel_system" type="system">
             <hardware>
@@ -24,4 +24,4 @@
             </joint>
         </ros2_control>
-    </xacro:macro> -->
+    </xacro:macro>
 </robot>
